File: cheroquee_kicad/cheroquee_kicad.kicad_pcb (KiCad board)
At the start: 2 copper layers, 67.3 x 78.7 mm, 26 parts, among them J1 Conn_01x05, Q1 2N3906, Q2 2N3906, Q3 2N3906, Q4 2N3906, Q5 2N3906, Q6 2N3906, Q7 2N3906, Q8 2N3906, U1 STP16, U2 STP16

Commit message: Update the protoboard
Parts:
- J1: value Conn_01x05 -> Conn_01x06; footprint Socket_Strips:Socket_Strip_Straight_1x05_Pitch2.54mm -> Socket_Strips:Socket_Strip_Straight_1x06_Pitch2.54mm
- U1, U2: footprint cheroquee:stp16_breakout -> cheroquee:stp16_breakout_alt
- moved U1 1.40 mm to (66.2, 58.5), turned to 0 degrees
- moved U2 0.18 mm to (66.2, 101.5), turned to 0 degrees
Connections:
- U1 pad 21: GNDREF -> ~OE
- U2 pad 21: GNDREF -> ~OE
Routing:
- net ~OE: track 0.00 -> 99.9 mm, vias 0 -> 1
- net +5V: track 62.9 -> 147.8 mm, vias 2 -> 10
- net GNDREF: track 145.2 -> 189.7 mm, vias 0 -> 1
- net C3: track 151.7 -> 109.1 mm
- net R3: track 54.2 -> 94.1 mm, vias 1 -> 0
- net R1: track 60.0 -> 97.3 mm
- net C4: track 93.3 -> 130.0 mm, vias 0 -> 1
- net R2: track 60.9 -> 92.6 mm, vias 0 -> 1
- net R4: track 44.0 -> 72.1 mm, vias 0 -> 1
- net CLK: track 77.4 -> 105.3 mm, vias 1 -> 0
- net R13: track 59.7 -> 84.8 mm
- net ST: track 86.3 -> 98.9 mm
- net SDI: track 93.7 -> 106.0 mm
- net en_C7: track 48.0 -> 60.3 mm
- net R16: track 32.1 -> 44.3 mm, vias 0 -> 1
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Other:
- board text added: "+5V"
- board text added: "CLK"
- board text added: "CS"
- board text added: "GND"
- board text added: "SDI"
- board text added: "~OE"
