File: cheroquee_kicad/cheroquee_kicad.sch (KiCad schematic (older format))
At the start: 26 parts, among them J1 Conn_01x05, Q1 2N3906, Q2 2N3906, Q3 2N3906, Q4 2N3906, Q5 2N3906, Q6 2N3906, Q7 2N3906, Q8 2N3906, U1 STP16, U2 STP16

Commit message: Update the protoboard
Parts:
- J1: value Conn_01x05 -> Conn_01x06; footprint Socket_Strips:Socket_Strip_Straight_1x05_Pitch2.54mm -> Socket_Strips:Socket_Strip_Straight_1x06_Pitch2.54mm; symbol Connector_Generic:Conn_01x05 -> Connector_Generic:Conn_01x06
- U1, U2: footprint cheroquee:stp16_breakout -> cheroquee:stp16_breakout_alt
Connections:
- net GNDREF: no longer U1.21 (~OE), U2.21 (~OE)
- new net ~OE: J1.6 (Pin_6), U1.21 (~OE), U2.21 (~OE)
Changed lines of the file:
@@
 F 0 "U1" H 1850 3800 60  0000 C BNN
 F 1 "STP16" H 1850 3700 60  0000 C BNN
-F 2 "cheroquee:stp16_breakout" H 1850 3050 60  0001 C CNN
+F 2 "cheroquee:stp16_breakout_alt" H 1850 3050 60  0001 C CNN
 F 3 "https://datasheets.maximintegrated.com/en/ds/MAX6969.pdf" H 1850 3050 60  0001 C CNN
 	1    1850 3050
@@
 F 0 "U2" H 1850 6200 60  0000 C BNN
 F 1 "STP16" H 1850 6100 60  0000 C BNN
-F 2 "cheroquee:stp16_breakout" H 1850 5450 60  0001 C CNN
+F 2 "cheroquee:stp16_breakout_alt" H 1850 5450 60  0001 C CNN
 F 3 "https://datasheets.maximintegrated.com/en/ds/MAX6969.pdf" H 1850 5450 60  0001 C CNN
 	1    1850 5450
@@
 Text GLabel 2250 2700 2    50   Input ~ 0
 SDO_1
-$Comp
-L power:GNDREF #PWR0108
-U 1 1 5C893ABA
-P 2800 2900
-F 0 "#PWR0108" H 2800 2650 50  0001 C CNN
-F 1 "GNDREF" H 2805 2727 50  0001 C CNN
-F 2 "" H 2800 2900 50  0001 C CNN
-F 3 "" H 2800 2900 50  0001 C CNN
-	1    2800 2900
-	1    0    0    -1
-$EndComp
-Wire Wire Line
-	2800 2900 2800 2800
-Wire Wire Line
-	2800 2800 2250 2800
 Text GLabel 1450 5000 0    50   Input ~ 0
 SDO_1
@@
 Text GLabel 1450 5100 0    50   Input ~ 0
 CLK
-$Comp
-L power:GNDREF #PWR0109
-U 1 1 5C8A1F2A
-P 2800 5250
-F 0 "#PWR0109" H 2800 5000 50  0001 C CNN
-F 1 "GNDREF" H 2805 5077 50  0001 C CNN
-F 2 "" H 2800 5250 50  0001 C CNN
-F 3 "" H 2800 5250 50  0001 C CNN
-	1    2800 5250
-	1    0    0    -1
-$EndComp
-Wire Wire Line
-	2800 5250 2800 5200
-Wire Wire Line
-	2250 5200 2800 5200
 Text GLabel 2250 5100 2    50   Input ~ 0
 SDO_2
@@
 ST
 $Comp
-L Connector_Generic:Conn_01x05 J1
+L Connector_Generic:Conn_01x06 J1
 U 1 1 5C8AD721
 P 4750 5100
 F 0 "J1" H 4830 5142 50  0000 L CNN
-F 1 "Conn_01x05" H 4830 5051 50  0000 L CNN
-F 2 "Socket_Strips:Socket_Strip_Straight_1x05_Pitch2.54mm" H 4750 5100 50  0001 C CNN
+F 1 "Conn_01x06" H 4830 5051 50  0000 L CNN
+F 2 "Socket_Strips:Socket_Strip_Straight_1x06_Pitch2.54mm" H 4750 5100 50  0001 C CNN
 F 3 "~" H 4750 5100 50  0001 C CNN
 	1    4750 5100
@@
 Wire Wire Line
 	4500 4600 4100 4600
+Text GLabel 2250 2800 2    50   Input ~ 0
+~OE
+Text GLabel 4100 5500 0    50   Input ~ 0
+~OE
+Text GLabel 2250 5200 2    50   Input ~ 0
+~OE
+Wire Wire Line
+	4100 5500 4200 5500
+Wire Wire Line
+	4200 5500 4200 5400
+Wire Wire Line
+	4200 5400 4550 5400
 $EndSCHEMATC
